Commit message: finish lab314

File: src/autolabor_description/urdf/autolabor_pro1.urdf (robot description, URDF)
Before this commit: robot autolabor_description, 1 links, 0 joints
Links:
- added link imu_link; visual cylinder length=0.02 radius=0.03
- added link velodyne; visual cylinder length=0.07 radius=0.05
Joints:
- added joint imu_link_joint: type fixed, parent base_link, child imu_link, origin xyz=0 0 1.4 rpy=0 0 0
- added joint velodyne_link_joint: type fixed, parent base_link, child velodyne, origin xyz=0 0 1.5 rpy=0 0 0

Commit message: add path demo

File: src/autolabor_description/urdf/autolabor_pro1.urdf (robot description, URDF)
Before this commit: robot autolabor_description, 3 links, 2 joints
Links:
- link imu_link: geometry visual box size=0.035 0.035 0.015
Joints:
- joint imu_link_joint: origin xyz=0 0 1.4 rpy=0 0 0 -> xyz=0 0 0 rpy=0 0 0
- joint velodyne_link_joint: origin xyz=0 0 1.5 rpy=0 0 0 -> xyz=0 0 0 rpy=0 0 0

Commit message: use hector and add ydlidar

File: src/autolabor_description/urdf/autolabor_pro1.urdf (robot description, URDF)
Before this commit: robot autolabor_description, 3 links, 2 joints
Links:
- added link imu; visual box size=0.035 0.035 0.015
- added link laser_frame; visual cylinder length=0.05 radius=0.03
Joints:
- added joint imu2_link_joint: type fixed, parent base_link, child imu, origin xyz=0 0 0 rpy=0 0 0
- added joint rplidar_link__joint: type fixed, parent base_link, child laser_frame, origin xyz=0 0 0 rpy=0 0 0

Commit message: add map tool

File: src/autolabor_description/urdf/autolabor_pro1.urdf (robot description, URDF)
Before this commit: robot autolabor_description, 5 links, 4 joints
Links:
- removed link laser_frame
- added link ydlidar_link; visual cylinder length=0.05 radius=0.03
Joints:
- removed joint rplidar_link__joint
- added joint ydlidar_link__joint: type fixed, parent base_link, child ydlidar_link, origin xyz=0 0 0 rpy=0 0 0
